Commit message: updated ros/gazebo example to work with gazebo>=7

File: examples/ros_example/src/p3dx_description/urdf/pioneer3dx.xacro (robot description, xacro)
@@ -92,5 +92,6 @@
 			<origin xyz="0 0 0" rpy="0 0 0" />
 			<geometry>
-				<box size="0 0 0" />
+				<!-- <box size="0.0 0.0 0.0" /> -->
+        		<box size="0.01 0.01 0.01"/>
 			</geometry>
 		</collision>
@@ -125,5 +126,6 @@
 			<origin xyz="0 0 0" rpy="0 0 0" />
 			<geometry>
-				<box size="0 0 0" />
+				<!-- <box size="0.0 0.0 0.0" /> -->
+				<box size="0.01 0.01 0.01" />
 			</geometry>
 		</collision>
@@ -188,5 +190,6 @@
 			<origin rpy="0 0 0" xyz="0 0 0" />
 			<geometry>
-				<box size="0 0 0" />
+				<!-- <box size="0.0 0.0 0.0" /> -->
+				<box size="0.01 0.01 0.01" />
 			</geometry>
 		</collision>

File: examples/ros_example/src/p3dx_description/urdf/pioneer3dx_wheel.xacro (robot description, xacro)
@@ -69,7 +69,7 @@
 			</visual>
 			<collision>
-				<origin xyz="0 0 0" rpy="0 0 0" />
+				<origin xyz="0.0 0.0 0.0" rpy="0.0 0.0 0.0" />
 				<geometry>
-					<box size="0 0 0" />
+					<box size="0.01 0.01 0.01" />
 				</geometry>
 			</collision>

Commit message: Adaption from Indigo/Gazebo2 to Melodic/Gazebo9. Proper visualization of robot color in melodic/Gazebo9 now.

File: examples/ros_example/src/p3dx_description/urdf/pioneer3dx.xacro (robot description, xacro)
@@ -29,5 +29,5 @@
 			<inertia ixx="1" ixy="0" ixz="0" iyy="1" iyz="0" izz="1" />
 		</inertial>
-		<visual name="base_visual">
+		<visual>
 			<origin xyz="-0.045 0 0.148" rpy="0 0 0" />
 			<geometry name="pioneer_geom">
@@ -52,5 +52,5 @@
 			<inertia ixx="1" ixy="0" ixz="0" iyy="1" iyz="0" izz="1" />
 		</inertial>
-		<visual name="base_visual">
+		<visual>
 			<origin xyz="0 0 0" rpy="0 0 0" />
 			<geometry name="top_geom">
@@ -80,5 +80,5 @@
 			<inertia ixx="0.01" ixy="0" ixz="0" iyy="0.01" iyz="0" izz="0.01" />
 		</inertial>
-		<visual name="base_visual">
+		<visual>
 			<origin xyz="0 0 0" rpy="0 0 0" />
 			<geometry name="pioneer_geom">
@@ -114,5 +114,5 @@
 				iyy="0.015218160428" iyz="-0.000004273467" izz="0.011763977943" />
 		</inertial>
-		<visual name="base_visual">
+		<visual>
 			<origin xyz="0 0 0" rpy="0 0 0" />
 			<geometry name="pioneer_geom">
@@ -148,5 +148,5 @@
 				iyy="0.015218160428" iyz="-0.000004273467" izz="0.011763977943" />
 		</inertial>
-		<visual name="base_visual">
+		<visual>
 			<origin xyz="0 0 0" rpy="0 0 0" />
 			<geometry name="pioneer_geom">
@@ -178,5 +178,5 @@
 			<inertia ixx="1" ixy="0" ixz="0" iyy="1" iyz="0" izz="1" />
 		</inertial>
-		<visual name="front_sonar_vis">
+		<visual>
 			<origin rpy="0 0 0" xyz="0 0 0" />
 			<geometry name="pioneer_geom">

File: examples/ros_example/src/p3dx_description/urdf/pioneer3dx_wheel.xacro (robot description, xacro)
@@ -18,5 +18,5 @@
 <robot xmlns:xacro="http://ros.org/wiki/xacro">
 	<!-- properties (constants) -->
-	<property name="M_PI" value="3.14159" />
+	<xacro:property name="M_PI" value="3.14159" />
 	<!-- right/left hubcap + wheel -->
 	<xacro:macro name="p3dx_wheel" params="suffix parent reflect">
@@ -29,5 +29,5 @@
 					iyz="0" izz="0.011763977943" />
 			</inertial>
-			<visual name="base_visual">
+			<visual>
 				<origin xyz="0 0 0" rpy="0 0 0" />
 				<geometry name="pioneer_geom">
@@ -59,5 +59,5 @@
 					iyz="0" izz="0.011763977943" />
 			</inertial>
-			<visual name="base_visual">
+			<visual>
 				<origin xyz="0 0 0" rpy="0 0 0" />
 				<geometry name="pioneer_geom">
